File: mysz.brd (EAGLE design)
At the start: 100 x 100.2 mm, 110 parts, among them IC1 ULN2003AD, IC2 MPU-9250, IC3 ACS712, IC4 ACS712, IC5 TLE9201SG, IC6 TLE9201SG, IC7 STM32F411RCT6, J2 7-188275-4, J3 7-188275-4, T1 BPX81, T2 BPX81, T3 BPX81, T4 BPX81, U1 V_REG_317-DPACK, U2 V_REG_317-DPACK, Y1 16Mhz

Commit message: Getting smaller
Parts:
- removed C1, C2: 33uF, Kell Ideas:PANASONIC_C
- removed C12, C14, C25: (no value), Kell Ideas:C0603K
- removed SJ1, SJ2: (no value), Kell Ideas:SJ
- removed U$11: DISPLAY-OLED-128X32, Kell Ideas:DISPLAY-OLED-128X32
- removed U1: V_REG_317-DPACK, Kell Ideas:V-REG_DPACK
- added R25, R26, R27, R28: 10k, Kell Ideas:R0603
- added R29, R30: (no value), Kell Ideas:R0603
- added T5, T6: BPX81, opto-trans-siemens:BPX81
- moved C27 119.5 mm to (38.7, -0.17), turned to 270 degrees
- moved R19 117.3 mm to (31.8, -4.09), turned to 180 degrees
- moved R14 115.6 mm to (33.8, -6.62)
- moved C29 111.1 mm to (24.8, 2.11), turned to 180 degrees
- moved R7 110.5 mm to (40.9, 3.38)
- moved C28 109.5 mm to (49.0, 2.07), turned to 180 degrees
- moved R13 107.7 mm to (40.9, 3.91), turned to 180 degrees
- moved C30 107.3 mm to (31.8, 3.32), turned to 180 degrees
- moved C7 100.2 mm to (-35.0, 30.0)
- moved C31 99.5 mm to (29.7, 11.2), turned to 270 degrees
- moved C3 96.1 mm to (132.0, 41.0)
- moved C15 93.4 mm to (118.6, -13.7)
- moved C17 93.4 mm to (122.9, -17.7)
- moved IC2 93.4 mm to (121.9, -13.7)
- moved R1 93.4 mm to (122.8, -10.6)
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Connections:
- net USART1_RX renamed RX
- net USART1_TX renamed TX
- removed net CZ1_OUT: R9.1, T1.C
- removed net CZ2_OUT: R10.1, T2.C
- removed net CZ3_OUT: R11.1, T3.C
- removed net CZ4_OUT: R12.1, T4.C
- removed net I2C3_SCL: IC7.41, R24.1
- removed net I2C3_SDA: IC7.40, R23.1
- removed net N$10: MOT2_A.1
- removed net N$11: MOT2_B.1
- removed net N$12: MOT1_B.1
- removed net N$21: S3.8
- removed net N$31: S3.6
- removed net N$34: S3.7
- removed net N$35: S3.5
- removed net N$9: MOT1_A.1
- new net MOT1_A: IC5.5, MOT1_A.1
- new net MOT1_B: IC5.7, MOT1_B.1
- new net MOT2_A: IC6.5, MOT2_A.1
- new net MOT2_B: IC6.7, MOT2_B.1
- new net SWIM: SV1.8
- new net SW_1: IC7.8, R25.1, S3.8
- new net SW_2: IC7.9, R26.1, S3.7
- new net SW_3: IC7.10, R27.1, S3.6
- new net SW_4: IC7.11, R28.1, S3.5
- net +3V3: now also R25.2, R26.2, R27.2, R28.2, R29.2, R30.2, SV1.3, SV1.4; no longer C25.1, U$11.2
- net +5V: now also SV1.1, SV1.2; no longer C14.1, C2.+, U1.4
- net BAT+: now also J1.+
- net DIST1: now also R9.1, T1.C
- net DIST2: now also R10.1, T2.C
- net DIST3: now also R11.1, T3.C
- net DIST4: now also R12.1, T4.C
- net DIST5: now also R29.1, T5.C
- net DIST6: now also R30.1, T6.C
- net GND: now also J1.-, SV1.5, SV1.6, T5.E, T6.E; no longer C1.-, C12.2, C14.2, C2.-, C25.2, U$11.1, U1.1
- net IR_LED_3: now also IC7.59; no longer IC7.60
- net IR_LED_4: now also IC7.58; no longer IC7.59
- net IR_LED_5: now also IC7.57; no longer IC7.58
- net IR_LED_6: now also IC7.56; no longer IC7.57
- net MOT1_DIR: now also IC7.36
- net MOT1_EN: now also IC7.35
- net MOT1_ENCODER_A: now also IC7.55; no longer IC7.14
- net MOT1_ENCODER_B: now also IC7.50; no longer IC7.15
- net MOT1_PWM: now also IC7.37
- net MOT2_DIR: now also IC7.39
- net MOT2_EN: now also IC7.34
- net MOT2_ENCODER_A: now also IC7.14; no longer IC7.55
- net MOT2_ENCODER_B: now also IC7.15; no longer IC7.50
- net MOT2_PWM: now also IC7.38
- net NRST: now also SV1.10
- net SCL: now also IC7.41, R24.1; no longer U$11.3
- net SDA: now also IC7.40, R23.1; no longer U$11.4
- net SWCLK: now also SV1.9
- net SWDIO: now also SV1.7
- net V+: no longer C1.+, C12.1, U1.3
Routing:
- net +3V3: track 14.9 -> 0.00 mm
- net RCC_OSC_IN: track 9.65 -> 0.00 mm
- net RCC_OSC_OUT: track 7.19 -> 0.00 mm
- net VDDA: track 6.93 -> 0.00 mm
- net IR_LED_6: track 6.08 -> 0.00 mm
- net IR_LED_1: track 5.89 -> 0.00 mm
- net IR_LED_5: track 5.76 -> 0.00 mm
- net IR_LED_2: track 5.57 -> 0.00 mm
- net IR_LED_4: track 5.44 -> 0.00 mm
- net IR_LED_3: track 5.25 -> 0.00 mm
- net I2C3_SDA: track 3.99 -> 0.00 mm
- net N$1: track 2.89 -> 0.00 mm
- net I2C3_SCL: track 2.29 -> 0.00 mm
- net GND: track 1.27 -> 0.00 mm
Other:
- board size 100 x 100.2 mm -> 69 x 63.7 mm

Commit message: Finished wiring
Parts:
- removed C10, C22: 33uF, Kell Ideas:PANASONIC_C
- removed C11, C13, C26, C28, C30, C33, C35: (no value), Kell Ideas:C0603K
- removed C15, C17: 100nF, Kell Ideas:C0603K
- removed IC1: ULN2003AD, uln-udn:SO16
- removed IC2: MPU-9250, Kell Ideas:QFN40P300X300X105-25N
- removed J1: (no value), Kell Ideas:DEANS
- removed J2, J3: 7-188275-4, Kell Ideas:7-188275-4
- removed LED1, LED13, LED2, LED3, LED4, LED6: (no value), led:Q62902-B155
- removed LED10, LED11, LED7, LED8, LED9: LEDCHIPLED_0603, Kell Ideas:CHIPLED_0603
- removed R1, R10, R11, R12, R13, R14, R15, R16, R17, R18, R19, R20, R21, R22, R29, R30, R9: (no value), Kell Ideas:R0603
- removed SG1: BUZZERPTH, SparkFun:BUZZER-12MM
- removed SV1: (no value), Kell Ideas:ML10
- removed T6: BPX81, opto-trans-siemens:BPX81
- removed U$12: WIRELESS-BLUETOOTH-HC-05, Kell Ideas:WIRELESS-BLUETOOTH-HC-05
- added JP2, POWER: (no value), pinhead:1X02
- added PROG-SWDIO: MICROMATCH-6, con-amp-micromatch:MICROMATCH-6
- added U$10, U$11, U$7, U$8, U$9: ADAFRUIT-VCNL4010, Kell Ideas:ADAFRUIT-VCNL4010
- added U$13, U$14: PRIV-AS5040, Kell Ideas:PRIV-AS5040
- IC3, IC4: value ACS712 -> ACS711
- JP1: device pinhead:1X04 -> pinhead:1X02
- S1: value TL32PO -> (none); device switch:TL3XPO -> SparkFun-Switches:SWITCH_SPDT_PTH_11.6X4.0MM
- T1, T2, T3, T4, T5: value BPX81 -> BC847; device opto-trans-siemens:BPX81 -> transistor:SOT23
- moved T5 127.4 mm to (7.62, 54.4), turned to 270 degrees
- moved C7 91.9 mm to (56.0, 17.5), turned to 0 degrees
- moved JP1 90.4 mm to (51.1, 7.62)
- moved C3 81.5 mm to (56.0, 11.5)
- moved C5 78.6 mm to (34.7, 6.21), turned to 180 degrees
- moved R28 76.6 mm to (14.2, 6.86), turned to 225 degrees
- moved C18 75.7 mm to (72.2, 17.6), turned to 90 degrees
- moved R2 75.6 mm to (50.8, 66.3), turned to 90 degrees
- moved R26 73.7 mm to (2.79, 13.7), turned to 225 degrees
- moved C24 73.4 mm to (33.1, 20.8)
- moved R25 72.9 mm to (5.08, 16.0), turned to 225 degrees
- moved R27 70.3 mm to (11.9, 4.57), turned to 225 degrees
- moved R4 70.1 mm to (68.5, 53.8), turned to 45 degrees
- moved C6 69.4 mm to (42.3, 6.76), turned to 270 degrees
- moved R5 67.0 mm to (63.8, 49.8)
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Connections:
- removed net +5V: C27.1, C29.1, IC3.8, IC4.8, R2.2, R21.2, R22.2, R3.2, R4.2, R5.2, SV1.1, SV1.2
- removed net AUX_CL: IC2.7
- removed net AUX_DA: IC2.21
- removed net BUZZER: SG1.+
- removed net DIST1: IC7.20, R9.1, T1.C
- removed net DIST2: IC7.21, R10.1, T2.C
- removed net DIST3: IC7.22, R11.1, T3.C
- removed net DIST4: IC7.23, R12.1, T4.C
- removed net DIST5: IC7.24, R29.1, T5.C
- removed net DIST6: IC7.25, R30.1, T6.C
- removed net FSYNC: IC2.11
- removed net INT: IC2.12
- removed net IR_LED_1: IC1.1, IC7.62
- removed net IR_LED_2: IC1.2, IC7.61
- removed net IR_LED_3: IC1.3, IC7.59
- removed net IR_LED_4: IC1.4, IC7.58
- removed net IR_LED_5: IC1.5, IC7.57
- removed net IR_LED_6: IC1.6, IC7.56
- removed net I_MOT1_5V: IC3.7, R7.2
- removed net I_MOT2_5V: IC4.7, R14.2
- removed net LED1: R20.1
- removed net LED2: R15.1
- removed net LED3: R16.1
- removed net LED4: R17.1
- removed net LED5: R18.1
- removed net N$1: C17.1, IC2.10
- removed net N$14: IC1.14, LED2.K
- removed net N$15: IC1.13, LED3.K
- removed net N$17: LED13.A, R2.1
- removed net N$18: LED1.A, R3.1
- removed net N$19: LED2.A, R4.1
- removed net N$20: LED3.A, R5.1
- removed net N$26: LED11.A, R20.2
- removed net N$27: C30.1, IC4.6
- removed net N$28: IC1.12, LED4.K
- removed net N$29: C28.1, IC3.6
- removed net N$30: IC1.11, LED6.K
- removed net N$32: LED4.A, R21.1
- removed net N$33: LED6.A, R22.1
- removed net NCS: IC2.22, R1.1
- new net BOOT0: IC7.60, JP1.2
- new net BOOT1: IC7.28, JP2.1
- new net DIST1_ON: IC7.56, R5.1
- new net DIST2_ON: IC7.57, R4.1
- new net DIST3_ON: IC7.58, R2.1
- new net DIST4_ON: IC7.59, R3.1
- new net DIST5_ON: IC7.61, R7.1
- new net MOT1_VS: IC3.3, IC3.4, IC5.4
- new net N$11: T3.2, U$9.VIN
- new net N$12: T4.2, U$10.VIN
- new net N$2: R2.2, T1.1
- new net N$9: T1.2, U$7.VIN
- net +3V3: now also C27.1, C29.1, IC3.8, IC4.8, JP1.1, PROG-SWDIO.1, T1.3, T2.3, T3.3, T4.3, T5.3, U$13.3V3, U$14.3V3; no longer C15.1, C22.+, C26.1, IC2.1, IC2.13, IC2.8, J2.1, J3.1, JP1.4, R1.2, R10.2, R11.2, R12.2, R29.2, R30.2, R9.2, SV1.3, SV1.4, U$12.5
- net BAT+: now also POWER.2; no longer J1.+
- net GND: now also JP2.2, POWER.1, PROG-SWDIO.2, S2.A2, U$10.GND, U$11.GND, U$13.GND, U$14.GND, U$7.GND, U$8.GND, U$9.GND; no longer C10.-, C11.2, C13.2, C15.2, C17.2, C22.-, C26.2, C28.2, C30.2, C33.2, C35.2, IC1.7, IC1.8, IC2.18, IC2.20, IC2.9, J1.-, J2.3, J3.3, JP1.3, LED10.C, LED11.C, LED7.C, LED8.C, LED9.C, R13.1, R19.1, S2.B1, SG1.-, SV1.5, SV1.6, T1.E, T2.E, T3.E, T4.E, T5.E, T6.E, U$12.4
- net I_MOT1: now also IC3.7; no longer R13.2, R7.1
- net I_MOT2: now also IC4.7; no longer R14.1, R19.2
- net MOT1_DIR: now also IC7.34; no longer IC7.36
- net MOT1_ENCODER_A: now also U$14.B; no longer J3.2
- net MOT1_ENCODER_B: now also U$14.A; no longer J3.4
- net MOT2_EN: now also IC7.36; no longer IC7.34
- net MOT2_ENCODER_A: now also U$13.B; no longer J2.2
- net MOT2_ENCODER_B: now also U$13.A; no longer J2.4
- net MOT2_VS: no longer IC3.3, IC3.4, IC5.4
- net N$13: now also T5.2, U$11.VIN; no longer IC1.15, LED1.K
- net N$3: now also R3.2, T2.1; no longer LED7.A, R18.2
- net N$4: now also R4.2, T3.1; no longer LED8.A, R17.2
- net N$5: now also R5.2, T4.1; no longer LED9.A, R16.2
- net N$6: now also R7.2, T5.1; no longer LED10.A, R15.2
- net N$8: now also T2.2, U$8.VIN; no longer IC1.16, LED13.K
- net NRST: now also PROG-SWDIO.6, S2.B1; no longer S2.A2, SV1.10
- net RX: no longer JP1.2, U$12.3
- net SCL: now also U$10.SCL, U$11.SCL, U$7.SCL, U$8.SCL, U$9.SCL; no longer IC2.23
- net SDA: now also U$10.SDA, U$11.SDA, U$7.SDA, U$8.SDA, U$9.SDA; no longer IC2.24
- net SWCLK: now also PROG-SWDIO.5; no longer SV1.9
- net SWDIO: now also PROG-SWDIO.3; no longer SV1.7
- net SWIM: now also PROG-SWDIO.4; no longer SV1.8
- net TX: no longer JP1.1, U$12.2
- net V+: now also S1.1; no longer C10.+, C11.1, C13.1, C33.1, C35.1, S1.3
Routing:
- net +3V3: track 0.00 -> 442.7 mm, vias 0 -> 9
- net SCL: track 0.00 -> 200.3 mm, vias 0 -> 6
- net SDA: track 0.00 -> 195.9 mm, vias 0 -> 4
- net V+: track 0.00 -> 87.7 mm, vias 0 -> 7
- net MOT1_ENCODER_A: track 0.00 -> 78.4 mm, vias 0 -> 2
- net MOT1_ENCODER_B: track 0.00 -> 77.8 mm, vias 0 -> 2
- net MOT2_DIR: track 0.00 -> 72.8 mm, vias 0 -> 3
- net DIST5_ON: track 0.00 -> 68.4 mm
- net DIST4_ON: track 0.00 -> 66.3 mm
- net DIST2_ON: track 0.00 -> 59.7 mm, vias 0 -> 2
- net DIST3_ON: track 0.00 -> 55.5 mm
- net MOT2_EN: track 0.00 -> 52.7 mm, vias 0 -> 1
- net DIST1_ON: track 0.00 -> 51.5 mm
- net MOT2_ENCODER_B: track 0.00 -> 51.1 mm, vias 0 -> 2
- net MOT2_ENCODER_A: track 0.00 -> 50.8 mm, vias 0 -> 2
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- added copper zone on layer 16, net GND
Other:
- board size 69 x 63.7 mm -> 74 x 70 mm
- board text added: "+"
- board text added: "GND"
