File: mysz.sch (EAGLE design)
At the start: 68 parts, among them IC1 ULN2003AD, T1 BPX81, T2 BPX81, T3 BPX81, T4 BPX81, U1 STM32F10XRXT6

Commit message: Added all planned sensors to schematic
Parts:
- removed CR1: 8MHz, crystal_scorpio:ABM7
- removed JP2: (no value), pinhead:PINHD-1X2
- removed JP3, JP4, JP5: (no value), pinhead:PINHD-1X4
- removed L1: 10uH, rcl:L-EUL2012C
- removed U$1: TB6621FNG, SparkFun:TB6621FNG
- added C22, C32, C34: 33uF, Kell Ideas:CPOL-EUC
- added C23, C24, C31, C36: 100nF, Kell Ideas:CAPACITOR_SMD_0603
- added C25, C26, C27, C28, C29, C30, C33, C35: (no value), Kell Ideas:CAPACITOR_SMD_0603
- added C8, C9: 18pF, Kell Ideas:CAPACITOR_SMD_0603
- added IC4: ACS712, Kell Ideas:ACS712
- added IC5, IC6: TLE9201SG, Kell Ideas:TLE9201SG
- added IC7: STM32F411RCT6, Kell Ideas:STM32F411RCT6
- added J1: (no value), Kell Ideas:BATTERY_CONN_DEANS
- added J2, J3: 7-188275-4, Kell Ideas:7-188275-4
- added L2: INDUCTOR-0603, Kell Ideas:INDUCTOR-0603
- added LED13, LED6: (no value), led:LEDB155
- added R13, R14, R19, R21, R22, R23, R24, R7: (no value), Kell Ideas:RESISTOR_SMD_0603
- added S3: SWS004, Kell Ideas:SWS004
- added SJ1, SJ2: (no value), Kell Ideas:SOLDER_JUMPER
- added SV1: (no value), Kell Ideas:ML10
- added U$11: DISPLAY-OLED-128X32, Kell Ideas:DISPLAY-OLED-128X32
- added U$12: WIRELESS-BLUETOOTH-HC-05, Kell Ideas:WIRELESS-BLUETOOTH-HC-05
- added U2: V_REG_317-DPACK, Kell Ideas:V_REG_317-DPACK
- added Y1: 16Mhz, Kell Ideas:CRYSTAL_SMALL"
- C1, C2, C3, C4: value 100nF -> 33uF; device resistor:C-EUC0603K -> Kell Ideas:CPOL-EUC
- C10: value 10uF -> 33uF; device rcl:CPOL-EUA/3216-18R -> Kell Ideas:CPOL-EUC
- C11: value 100nF -> (none); device resistor:C-EUC0603K -> Kell Ideas:CAPACITOR_SMD_0603
- C12, C14, C16, C18: value 100nF -> (none); device rcl:C-EUC0603 -> Kell Ideas:CAPACITOR_SMD_0603
- C13: value 33uF -> (none); device rcl:CPOL-EU153CLV-1010 -> Kell Ideas:CAPACITOR_SMD_0603
- C15: value 47uF -> 100nF; device rcl:CPOL-EU153CLV-1010 -> Kell Ideas:CAPACITOR_SMD_0603
- C17: value 10uF -> 100nF; device rcl:CPOL-EU153CLV-1010 -> Kell Ideas:CAPACITOR_SMD_0603
- C19, C5, C6: device resistor:C-EUC0603K -> Kell Ideas:CAPACITOR_SMD_0603
- C20, C21: value 20pF -> 100nF; device resistor:C-EUC0603K -> Kell Ideas:CAPACITOR_SMD_0603
- C7: value 100uF -> 33uF; device rcl:CPOL-EU153CLV-1010 -> Kell Ideas:CPOL-EUC
- IC2: value (none) -> MPU-9250; device SparkFun:V_REG_LM1117SOT223 -> Kell Ideas:MPU-9250
- IC3: value (none) -> ACS712; device SparkFun:V_REG_LM1117SOT223 -> Kell Ideas:ACS712
- LED1, LED2, LED3, LED4: device led:LED5MM -> led:LEDB155
- LED10, LED11, LED7, LED8, LED9: value (none) -> LEDCHIPLED_0603; device led:LEDCHIPLED_0603 -> Kell Ideas:LEDCHIPLED_0603
- R1, R8: value 100k -> (none); device resistor:R-EU_R0603 -> Kell Ideas:RESISTOR_SMD_0603
- R10, R11, R12, R9: value 22k -> (none); device rcl:R-EU_R0603 -> Kell Ideas:RESISTOR_SMD_0603
- R15, R16, R17, R18, R20: value 680R -> (none); device resistor:R-EU_R0603 -> Kell Ideas:RESISTOR_SMD_0603
- R2, R3, R4, R5: value 100R -> (none); device rcl:R-EU_R0603 -> Kell Ideas:RESISTOR_SMD_0603
- R6: value 1.1k -> (none); device resistor:R-EU_R0603 -> Kell Ideas:RESISTOR_SMD_0603
- S2: value SWITCH-MOMENTARY-2-SMD-1101NE -> MOMENTARY-SWITCH-SPST-SMD-6.2MM_TALL; device SparkFun:SWITCH-MOMENTARY-2-SMD-1101NE -> Kell Ideas:MOMENTARY-SWITCH-SPST-SMD-6.2MM_TALL
- U1: value STM32F10XRXT6 -> V_REG_317-DPACK; device stm32:STM32F10XRXT6 -> Kell Ideas:V_REG_317-DPACK
Connections:
- removed net CZ1: IC1.I1, U1PORTA_H.PA11
- removed net CZ2: IC1.I2, U1PORTA_H.PA10
- removed net CZ3: IC1.I3, U1PORTA_H.PA9
- removed net CZ4: IC1.I4, U1PORTA_H.PA8
- removed net ENC1_A: JP4.3, U1PORTA_L.PA1
- removed net ENC1_B: JP4.2, U1PORTA_L.PA2
- removed net ENC2_A: JP5.3, U1PORTA_L.PA6
- removed net ENC2_B: JP5.2, U1PORTA_L.PA7
- removed net IN1_A: U$1.AIN1, U1PORTC_H.PC13
- removed net IN1_B: U$1.BIN1, U1PORTC_H.PC14
- removed net IN2_A: U$1.AIN2, U1PORTB_H.PB9
- removed net IN2_B: U$1.BIN2, U1PORTC_H.PC15
- removed net N$2: C5.1, L1.2, U1AN_POWER.VDDA
- removed net N$23: C20.1, CR1.P$2, U1PORTD/OSC.PD0/OSC<=
- removed net N$24: C21.1, CR1.P$1, U1PORTD/OSC.PD1/OSC=>
- removed net PWM_A: U$1.PWMA, U1PORTB_L.PB7
- removed net PWM_B: U$1.PWMB, U1PORTB_L.PB6
- removed net RESET: C19.1, R8.1, S2.1, U1RESET.NRST
- removed net RX: JP1.2, U1PORTB_H.PB11
- removed net TX: JP1.3, U1PORTB_H.PB10
- new net AUX_CL: IC2.AUX_CL
- new net AUX_DA: IC2.AUX_DA
- new net DIST1: IC7.PA4
- new net DIST2: IC7.PA5
- new net DIST3: IC7.PA6
- new net DIST4: IC7.PA7
- new net DIST5: IC7.PC4
- new net DIST6: IC7.PC5
- new net FSYNC: IC2.FSYNC
- new net I2C3_SCL: IC7.PA8, R24.1
- new net I2C3_SDA: IC7.PC9, R23.1
- new net INT: IC2.INT
- new net IR_LED_1: IC1.I1, IC7.PB9
- new net IR_LED_2: IC1.I2, IC7.PB8
- new net IR_LED_3: IC1.I3, IC7.BOOT0
- new net IR_LED_4: IC1.I4, IC7.PB7
- new net IR_LED_5: IC1.I5, IC7.PB6
- new net IR_LED_6: IC1.I6, IC7.PB5
- new net I_MOT1: IC7.PB1, R13.2, R7.1
- new net I_MOT1_5V: IC3.VIOUT, R7.2
- new net I_MOT2: IC7.PB0, R14.1, R19.2
- new net I_MOT2_5V: IC4.VIOUT, R14.2
- new net MOT1_DIR: IC5.DIR
- new net MOT1_EN: IC5.DIS
- new net MOT1_ENCODER_A: IC7.PA0, J3.2
- new net MOT1_ENCODER_B: IC7.PA1, J3.4
- new net MOT1_PWM: IC5.PWM
- new net MOT1_SO: IC5.SO
- new net MOT2_DIR: IC6.DIR
- new net MOT2_EN: IC6.DIS
- new net MOT2_ENCODER_A: IC7.PB3, J2.2
- new net MOT2_ENCODER_B: IC7.PA15, J2.4
- new net MOT2_PWM: IC6.PWM
- new net MOT2_SO: IC6.SO
- new net MOT2_VS: IC3.IP-_1, IC3.IP-_2, IC4.IP-_1, IC4.IP-_2, IC5.VS, IC6.VS
- new net N$21: S3.8
- new net N$27: C30.1, IC4.FILTER
- new net N$28: IC1.O5, LED4.C
- new net N$29: C28.1, IC3.FILTER
- new net N$30: IC1.O6, LED6.C
- new net N$31: S3.6
- new net N$32: LED4.A, R21.1
- new net N$33: LED6.A, R22.1
- new net N$34: S3.7
- new net N$35: S3.5
- new net NCS: IC2.NCS, R1.1
- new net NRST: C19.1, IC7.NRST, R8.1, S2.2
- new net RCC_OSC_IN: C8.2, IC7.PH0-OSC_IN, Y1.2
- new net RCC_OSC_OUT: C9.2, IC7.PH1-OSC_OUT, Y1.1
- new net SCL: IC2.SCL/SCLK, U$11.SCL
- new net SDA: IC2.SDA/SDI, U$11.SDA
- new net USART1_RX: IC7.PA10, JP1.2, U$12.TX
- new net USART1_TX: IC7.PA9, JP1.1, U$12.RX
- new net VDDA: C21.1, IC7.VDDA/VREF+, L2.2
- net +3V3: now also C15.1, C20.1, C22.+, C23.1, C24.1, C25.1, C26.1, C31.1, C36.1, C4.+, C5.1, IC2.VDD, IC2.VDDIO, IC5.VSO, IC6.VSO, IC7.VDD_1, IC7.VDD_2, IC7.VDD_3, IC7.VDD_4, J2.1, J3.1, L2.1, R1.2, R23.2, R24.2, U$11.VCC, U$12.+5V, U2.OUT; no longer C1.1, C17.+, C2.1, C3.1, C4.1, IC3.OUT, IC3.OUT@1, JP3.4, JP4.4, JP5.4, L1.1, U$1.STBY, U$1.VCC, U1AN_POWER.VBAT, U1POWER.VDD_1, U1POWER.VDD_2, U1POWER.VDD_3, U1POWER.VDD_4
- net +5V: now also C2.+, C27.1, C29.1, IC3.VCC, IC4.VCC, R21.2, R22.2, U1.OUT; no longer C13.+, IC2.OUT, IC2.OUT@1
- net BAT+: no longer JP2.1
- net BUZZER: no longer U1PORTB_H.PB8
- net CZ1_OUT: no longer U1PORTC_L.PC0
- net CZ2_OUT: no longer U1PORTC_L.PC1
- net CZ3_OUT: no longer U1PORTC_L.PC2
- net CZ4_OUT: no longer U1PORTC_L.PC3
- net GND: now also C1.-, C13.2, C15.2, C17.2, C2.-, C22.-, C23.2, C24.2, C25.2, C26.2, C27.2, C28.2, C29.2, C3.-, C30.2, C31.2, C32.-, C33.2, C34.-, C35.2, C36.2, C4.-, C8.1, C9.1, IC2.AD0/SDO, IC2.GND, IC3.GND, IC4.GND, IC5.CS_N, IC5.GND@1, IC5.GND@2, IC5.SCK, IC5.SI, IC6.CS_N, IC6.GND@1, IC6.GND@2, IC6.SCK, IC6.SI, IC7.VSSA/VREF-, IC7.VSS_1, IC7.VSS_2, IC7.VSS_3, IC7.VSS_4, J2.3, J3.3, JP1.3, R13.1, R19.1, S2.1, S3.1, S3.2, S3.3, S3.4, U$11.GND, U$12.GND, U1.ADJ, U2.ADJ; no longer C1.2, C13.-, C15.-, C17.-, C2.2, C3.2, C4.2, IC1.I5, IC1.I6, IC2.ADJ, IC3.ADJ, JP1.1, JP2.2, JP3.1, JP4.1, JP5.1, R1.2, S2.2, U$1.GND, U$1.PGND1@3, U$1.PGND1@4, U$1.PGND2@10, U$1.PGND2@9, U1AN_POWER.VSSA, U1POWER.VSS_1, U1POWER.VSS_2, U1POWER.VSS_3, U1POWER.VSS_4
- net LED1: no longer U1PORTC_H.PC8
- net LED2: no longer U1PORTC_H.PC9
- net LED3: no longer U1PORTC_H.PC10
- net LED4: no longer U1PORTC_H.PC11
- net LED5: no longer U1PORTC_H.PC12
- net N$1: now also C17.1, IC2.REGOUT; no longer R1.1, U1RESET.BOOT0
- net N$10: no longer U$1.A02@5, U$1.A02@6
- net N$11: no longer U$1.B02@7, U$1.B02@8
- net N$12: no longer U$1.B01@11, U$1.B01@12
- net N$13: now also LED1.C; no longer LED2.C
- net N$14: now also LED2.C; no longer LED3.C
- net N$15: now also LED3.C; no longer LED4.C
- net N$17: now also LED13.A; no longer LED1.A
- net N$18: now also LED1.A; no longer LED2.A
- net N$19: now also LED2.A; no longer LED3.A
- net N$20: now also LED3.A; no longer LED4.A
- net N$8: now also LED13.C; no longer LED1.C
- net N$9: no longer U$1.A01@1, U$1.A01@2
- net SWCLK: now also IC7.PA14; no longer JP3.2, U1PORTA_H.PA14
- net SWDIO: now also IC7.PA13; no longer JP3.3, U1PORTA_H.PA13
- net V+: now also C1.+, C13.1, C3.+, C32.+, C33.1, C34.+, C35.1, IC3.IP+_1, IC3.IP+_2, IC4.IP+_1, IC4.IP+_2, U1.IN, U2.IN; no longer C15.+, IC2.IN, IC3.IN, U$1.VM1, U$1.VM2, U$1.VM3
Other:
- moved on the sheet: C10, C11, C12, C14, C16, C18, C19, C20, C21, C5, C6, C7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

Commit message: Getting smaller
Parts:
- removed C1, C2: 33uF, Kell Ideas:CPOL-EUC
- removed C12, C14, C25: (no value), Kell Ideas:CAPACITOR_SMD_0603
- removed SJ1, SJ2: (no value), Kell Ideas:SOLDER_JUMPER
- removed U$11: DISPLAY-OLED-128X32, Kell Ideas:DISPLAY-OLED-128X32
- removed U1: V_REG_317-DPACK, Kell Ideas:V_REG_317-DPACK
- added R25, R26, R27, R28: 10k, Kell Ideas:RESISTOR_SMD_0603
- added R29, R30: (no value), Kell Ideas:RESISTOR_SMD_0603
- added T5, T6: BPX81, opto-trans-siemens:BPX81
Connections:
- net USART1_RX renamed RX
- net USART1_TX renamed TX
- removed net CZ1_OUT: R9.1, T1.C
- removed net CZ2_OUT: R10.1, T2.C
- removed net CZ3_OUT: R11.1, T3.C
- removed net CZ4_OUT: R12.1, T4.C
- removed net I2C3_SCL: IC7.PA8, R24.1
- removed net I2C3_SDA: IC7.PC9, R23.1
- removed net N$10: MOT2_A.1
- removed net N$11: MOT2_B.1
- removed net N$12: MOT1_B.1
- removed net N$21: S3.8
- removed net N$31: S3.6
- removed net N$34: S3.7
- removed net N$35: S3.5
- removed net N$9: MOT1_A.1
- new net MOT1_A: IC5.OUT1, MOT1_A.1
- new net MOT1_B: IC5.OUT2, MOT1_B.1
- new net MOT2_A: IC6.OUT1, MOT2_A.1
- new net MOT2_B: IC6.OUT2, MOT2_B.1
- new net SWIM: SV1.8
- new net SW_1: IC7.PC0, R25.1, S3.8
- new net SW_2: IC7.PC1, R26.1, S3.7
- new net SW_3: IC7.PC2, R27.1, S3.6
- new net SW_4: IC7.PC3, R28.1, S3.5
- net +3V3: now also R25.2, R26.2, R27.2, R28.2, R29.2, R30.2, SV1.3, SV1.4; no longer C25.1, U$11.VCC
- net +5V: now also SV1.1, SV1.2; no longer C14.1, C2.+, U1.OUT
- net BAT+: now also J1.+
- net DIST1: now also R9.1, T1.C
- net DIST2: now also R10.1, T2.C
- net DIST3: now also R11.1, T3.C
- net DIST4: now also R12.1, T4.C
- net DIST5: now also R29.1, T5.C
- net DIST6: now also R30.1, T6.C
- net GND: now also J1.-, SV1.5, SV1.6, T5.E, T6.E; no longer C1.-, C12.2, C14.2, C2.-, C25.2, U$11.GND, U1.ADJ
- net IR_LED_3: now also IC7.PB7; no longer IC7.BOOT0
- net IR_LED_4: now also IC7.PB6; no longer IC7.PB7
- net IR_LED_5: now also IC7.PB5; no longer IC7.PB6
- net IR_LED_6: now also IC7.PB4; no longer IC7.PB5
- net MOT1_DIR: now also IC7.PB15
- net MOT1_EN: now also IC7.PB14
- net MOT1_ENCODER_A: now also IC7.PB3; no longer IC7.PA0
- net MOT1_ENCODER_B: now also IC7.PA15; no longer IC7.PA1
- net MOT1_PWM: now also IC7.PC6
- net MOT2_DIR: now also IC7.PC8
- net MOT2_EN: now also IC7.PB13
- net MOT2_ENCODER_A: now also IC7.PA0; no longer IC7.PB3
- net MOT2_ENCODER_B: now also IC7.PA1; no longer IC7.PA15
- net MOT2_PWM: now also IC7.PC7
- net NRST: now also SV1.10
- net SCL: now also IC7.PA8, R24.1; no longer U$11.SCL
- net SDA: now also IC7.PC9, R23.1; no longer U$11.SDA
- net SWCLK: now also SV1.9
- net SWDIO: now also SV1.7
- net V+: no longer C1.+, C12.1, U1.IN

Commit message: Finished wiring
Parts:
- removed C10, C22: 33uF, Kell Ideas:CPOL-EUC
- removed C11, C13, C26, C28, C30, C33, C35: (no value), Kell Ideas:CAPACITOR_SMD_0603
- removed C15, C17: 100nF, Kell Ideas:CAPACITOR_SMD_0603
- removed IC1: ULN2003AD, uln-udn:ULN2003AD
- removed IC2: MPU-9250, Kell Ideas:MPU-9250
- removed J1: (no value), Kell Ideas:BATTERY_CONN_DEANS
- removed J2, J3: 7-188275-4, Kell Ideas:7-188275-4
- removed LED1, LED13, LED2, LED3, LED4, LED6: (no value), led:LEDB155
- removed LED10, LED11, LED7, LED8, LED9: LEDCHIPLED_0603, Kell Ideas:LEDCHIPLED_0603
- removed R1, R10, R11, R12, R13, R14, R15, R16, R17, R18, R19, R20, R21, R22, R29, R30, R9: (no value), Kell Ideas:RESISTOR_SMD_0603
- removed SG1: BUZZERPTH, SparkFun:BUZZERPTH
- removed SV1: (no value), Kell Ideas:ML10
- removed T6: BPX81, opto-trans-siemens:BPX81
- removed U$12: WIRELESS-BLUETOOTH-HC-05, Kell Ideas:WIRELESS-BLUETOOTH-HC-05
- added JP2, POWER: (no value), pinhead:PINHD-1X2
- added PROG-SWDIO: MICROMATCH-6, con-amp-micromatch:MICROMATCH-6
- added U$10, U$11, U$7, U$8, U$9: ADAFRUIT-VCNL4010, Kell Ideas:ADAFRUIT-VCNL4010
- added U$13, U$14: PRIV-AS5040, Kell Ideas:PRIV-AS5040
- IC3, IC4: value ACS712 -> ACS711
- JP1: device pinhead:PINHD-1X4 -> pinhead:PINHD-1X2
- S1: value TL32PO -> (none); device switch:TL32PO -> SparkFun-Switches:SWITCH-SPDT-PTH-11.6X4.0MM
- T1, T2, T3, T4, T5: value BPX81 -> BC847; device opto-trans-siemens:BPX81 -> transistor:BC847
Connections:
- removed net +5V: C27.1, C29.1, IC3.VCC, IC4.VCC, R2.2, R21.2, R22.2, R3.2, R4.2, R5.2, SV1.1, SV1.2
- removed net AUX_CL: IC2.AUX_CL
- removed net AUX_DA: IC2.AUX_DA
- removed net BUZZER: SG1.1
- removed net DIST1: IC7.PA4, R9.1, T1.C
- removed net DIST2: IC7.PA5, R10.1, T2.C
- removed net DIST3: IC7.PA6, R11.1, T3.C
- removed net DIST4: IC7.PA7, R12.1, T4.C
- removed net DIST5: IC7.PC4, R29.1, T5.C
- removed net DIST6: IC7.PC5, R30.1, T6.C
- removed net FSYNC: IC2.FSYNC
- removed net INT: IC2.INT
- removed net IR_LED_1: IC1.I1, IC7.PB9
- removed net IR_LED_2: IC1.I2, IC7.PB8
- removed net IR_LED_3: IC1.I3, IC7.PB7
- removed net IR_LED_4: IC1.I4, IC7.PB6
- removed net IR_LED_5: IC1.I5, IC7.PB5
- removed net IR_LED_6: IC1.I6, IC7.PB4
- removed net I_MOT1_5V: IC3.VIOUT, R7.2
- removed net I_MOT2_5V: IC4.VIOUT, R14.2
- removed net LED1: R20.1
- removed net LED2: R15.1
- removed net LED3: R16.1
- removed net LED4: R17.1
- removed net LED5: R18.1
- removed net N$1: C17.1, IC2.REGOUT
- removed net N$14: IC1.O3, LED2.C
- removed net N$15: IC1.O4, LED3.C
- removed net N$17: LED13.A, R2.1
- removed net N$18: LED1.A, R3.1
- removed net N$19: LED2.A, R4.1
- removed net N$20: LED3.A, R5.1
- removed net N$26: LED11.A, R20.2
- removed net N$27: C30.1, IC4.FILTER
- removed net N$28: IC1.O5, LED4.C
- removed net N$29: C28.1, IC3.FILTER
- removed net N$30: IC1.O6, LED6.C
- removed net N$32: LED4.A, R21.1
- removed net N$33: LED6.A, R22.1
- removed net NCS: IC2.NCS, R1.1
- new net BOOT0: IC7.BOOT0, JP1.2
- new net BOOT1: IC7.PB2, JP2.1
- new net DIST1_ON: IC7.PB4, R5.1
- new net DIST2_ON: IC7.PB5, R4.1
- new net DIST3_ON: IC7.PB6, R2.1
- new net DIST4_ON: IC7.PB7, R3.1
- new net DIST5_ON: IC7.PB8, R7.1
- new net MOT1_VS: IC3.IP-_1, IC3.IP-_2, IC5.VS
- new net N$11: T3.E, U$9.VIN
- new net N$12: T4.E, U$10.VIN
- new net N$2: R2.2, T1.B
- new net N$9: T1.E, U$7.VIN
- net +3V3: now also C27.1, C29.1, IC3.VCC, IC4.VCC, JP1.1, PROG-SWDIO-1.S, T1.C, T2.C, T3.C, T4.C, T5.C, U$13.3V3, U$14.3V3; no longer C15.1, C22.+, C26.1, IC2.VDD, IC2.VDDIO, J2.1, J3.1, JP1.4, R1.2, R10.2, R11.2, R12.2, R29.2, R30.2, R9.2, SV1.3, SV1.4, U$12.+5V
- net BAT+: now also POWER.2; no longer J1.+
- net GND: now also JP2.2, POWER.1, PROG-SWDIO-2.S, U$10.GND, U$11.GND, U$13.GND, U$14.GND, U$7.GND, U$8.GND, U$9.GND; no longer C10.-, C11.2, C13.2, C15.2, C17.2, C22.-, C26.2, C28.2, C30.2, C33.2, C35.2, IC1.GND, IC1.I7, IC2.AD0/SDO, IC2.GND, J1.-, J2.3, J3.3, JP1.3, LED10.C, LED11.C, LED7.C, LED8.C, LED9.C, R13.1, R19.1, SG1.2, SV1.5, SV1.6, T1.E, T2.E, T3.E, T4.E, T5.E, T6.E, U$12.GND
- net I_MOT1: now also IC3.VIOUT; no longer R13.2, R7.1
- net I_MOT2: now also IC4.VIOUT; no longer R14.1, R19.2
- net MOT1_DIR: now also IC7.PB13; no longer IC7.PB15
- net MOT1_ENCODER_A: now also U$14.B; no longer J3.2
- net MOT1_ENCODER_B: now also U$14.A; no longer J3.4
- net MOT2_EN: now also IC7.PB15; no longer IC7.PB13
- net MOT2_ENCODER_A: now also U$13.B; no longer J2.2
- net MOT2_ENCODER_B: now also U$13.A; no longer J2.4
- net MOT2_VS: no longer IC3.IP-_1, IC3.IP-_2, IC5.VS
- net N$13: now also T5.E, U$11.VIN; no longer IC1.O2, LED1.C
- net N$3: now also R3.2, T2.B; no longer LED7.A, R18.2
- net N$4: now also R4.2, T3.B; no longer LED8.A, R17.2
- net N$5: now also R5.2, T4.B; no longer LED9.A, R16.2
- net N$6: now also R7.2, T5.B; no longer LED10.A, R15.2
- net N$8: now also T2.E, U$8.VIN; no longer IC1.O1, LED13.C
- net NRST: now also PROG-SWDIO-6.S; no longer SV1.10
- net RX: no longer JP1.2, U$12.TX
- net SCL: now also U$10.SCL, U$11.SCL, U$7.SCL, U$8.SCL, U$9.SCL; no longer IC2.SCL/SCLK
- net SDA: now also U$10.SDA, U$11.SDA, U$7.SDA, U$8.SDA, U$9.SDA; no longer IC2.SDA/SDI
- net SWCLK: now also PROG-SWDIO-5.S; no longer SV1.9
- net SWDIO: now also PROG-SWDIO-3.S; no longer SV1.7
- net SWIM: now also PROG-SWDIO-4.S; no longer SV1.8
- net TX: no longer JP1.1, U$12.RX
- net V+: now also S1.O; no longer C10.+, C11.1, C13.1, C33.1, C35.1, S1.S
